Commit message: Imported upstream version '2.9.0' of 'upstream'

File: omni_base_description/robots/omni_base.urdf.xacro (robot description, xacro)
@@ -20,4 +20,6 @@
   <!-- false, true-->
   <xacro:arg name="add_on_module" default="no-add-on"/>
+  <!-- no-camera, realsense-d435, realsense-d435i -->
+  <xacro:arg name="camera_model" default="no-camera"/>
   <!-- Execution env config -->
   <xacro:arg name="use_sim_time" default="false"/>
@@ -30,4 +32,5 @@
   <xacro:property name="rear_laser_model" value="$(arg rear_laser_model)" />
   <xacro:property name="add_on_module" value="$(arg add_on_module)"/>
+  <xacro:property name="camera_model" value="$(arg camera_model)" />
   <!-- HW configuration check -->
   <xacro:if value="${front_laser_model not in ['no-laser', 'sick-551', 'sick-561', 'sick-571', 'hokuyo']}">
@@ -37,6 +40,9 @@
     <xacro:wrong_laser_model/>
   </xacro:if>
-  <xacro:if value="${add_on_module not in ['no-add-on', 'rgbd-sensors']}">
+  <xacro:if value="${add_on_module not in ['no-add-on', 'cobra']}">
     <xacro:wrong_add_on_module/>
+  </xacro:if>
+  <xacro:if value="${camera_model not in ['no-camera', 'realsense-d435', 'realsense-d435i']}">
+    <xacro:wrong_camera_model/>
   </xacro:if>
   <!-- Execution env configuration -->
@@ -49,5 +55,5 @@
   <xacro:include filename="$(find omni_base_description)/urdf/base/base_sensors.urdf.xacro" />
   <!-- RGBD Sensors -->
-  <xacro:if value="${add_on_module == 'rgbd-sensors'}">
+  <xacro:if value="${add_on_module == 'cobra'}">
     <xacro:include filename="$(find omni_base_description)/urdf/cameras_add_on/cameras_add_on.urdf.xacro" />
   </xacro:if>
@@ -63,5 +69,5 @@
   <xacro:base_sensors name="base" front_laser_model="$(arg front_laser_model)" rear_laser_model="$(arg rear_laser_model)"/>
   <!-- RGBD Sensors -->
-  <xacro:if value="${add_on_module == 'rgbd-sensors'}">
+  <xacro:if value="${add_on_module == 'cobra'}">
     <xacro:cameras_add_on name="cameras_add_on" parent="base_link"/>
   </xacro:if>

File: omni_base_description/urdf/base/base_sensors.urdf.xacro (robot description, xacro)
@@ -65,11 +65,5 @@
         <origin xyz="0 0 ${laser_height}" rpy="0 0 0" />
     </joint>
-    <link name="virtual_${name}_laser_link">
-        <inertial>
-            <origin xyz="0 0 0" rpy="0 0 0"/>
-            <mass value="0.0001" />
-            <inertia ixx="0.0001"  ixy="0"  ixz="0" iyy="0.0001" iyz="0" izz="0.0001" />
-        </inertial>
-    </link>
+    <link name="virtual_${name}_laser_link"/>
     <!-- IMU -->
     <xacro:imu_sensor name="${name}_imu" parent="${name}_link" update_rate="100.0">

File: omni_base_description/urdf/sensors/courier.urdf.xacro (robot description, xacro)
@@ -26,37 +26,71 @@
   <xacro:property name="roof_rgbd_y" value="0.0"/>
   <xacro:property name="roof_rgbd_Y" value="0.0"/>
-  <!-- INCLUDES -->
-  <xacro:include filename="$(find realsense2_description)/urdf/_d435.urdf.xacro" />
   <!-- base/roof RGBD calibratable characteristics -->
   <!-- spec = rgbd_z, rgbd_R and rgbd_P -->
   <xacro:include filename="${calibration_path}/urdf/cameras_add_on/base_omni_base_calib.urdf.xacro"/>
   <xacro:include filename="$(find pal_urdf_utils)/urdf/deg_to_rad.urdf.xacro" />
-  <!-- RGBD base -->
-  <xacro:sensor_d435
-    name="base_rgbd_camera"
-    parent="base_link"
-    topics_ns="base_rgbd_camera"
-    use_nominal_extrinsics="${use_sim_time}">
-    <origin
-        xyz="${base_rgbd_x}
-             ${base_rgbd_y}
-             ${base_rgbd_z}"
-        rpy="${base_rgbd_R * deg_to_rad}
-             ${base_rgbd_P * deg_to_rad}
-             ${base_rgbd_Y * deg_to_rad}"/>
-  </xacro:sensor_d435>
-  <!-- RGBD roof -->
-  <xacro:sensor_d435
-    name="roof_rgbd_camera"
-    parent="base_link"
-    topics_ns="roof_rgbd_camera"
-    use_nominal_extrinsics="${use_sim_time}">
-    <origin
-        xyz="${roof_rgbd_x}
-             ${roof_rgbd_y}
-             ${roof_rgbd_z}"
-        rpy="${roof_rgbd_R * deg_to_rad}
-             ${roof_rgbd_P * deg_to_rad}
-             ${roof_rgbd_Y * deg_to_rad}"/>
-  </xacro:sensor_d435>
+  <xacro:if value="${camera_model == 'realsense-d435'}">
+    <!-- INCLUDES -->
+    <xacro:include filename="$(find realsense2_description)/urdf/_d435.urdf.xacro" />
+    <!-- RGBD base -->
+    <xacro:sensor_d435
+      name="base_rgbd_camera"
+      parent="base_link"
+      topics_ns="base_rgbd_camera"
+      use_nominal_extrinsics="${use_sim_time}">
+      <origin
+          xyz="${base_rgbd_x}
+              ${base_rgbd_y}
+              ${base_rgbd_z}"
+          rpy="${base_rgbd_R * deg_to_rad}
+              ${base_rgbd_P * deg_to_rad}
+              ${base_rgbd_Y * deg_to_rad}"/>
+    </xacro:sensor_d435>
+    <!-- RGBD roof -->
+    <xacro:sensor_d435
+      name="roof_rgbd_camera"
+      parent="base_link"
+      topics_ns="roof_rgbd_camera"
+      use_nominal_extrinsics="${use_sim_time}">
+      <origin
+          xyz="${roof_rgbd_x}
+              ${roof_rgbd_y}
+              ${roof_rgbd_z}"
+          rpy="${roof_rgbd_R * deg_to_rad}
+              ${roof_rgbd_P * deg_to_rad}
+              ${roof_rgbd_Y * deg_to_rad}"/>
+    </xacro:sensor_d435>
+  </xacro:if>
+  <xacro:if value="${camera_model == 'realsense-d435i'}">
+    <!-- INCLUDES -->
+    <xacro:include filename="$(find realsense2_description)/urdf/_d435i.urdf.xacro" />
+    <!-- RGBD base -->
+    <xacro:sensor_d435i
+      name="base_rgbd_camera"
+      parent="base_link"
+      topics_ns="base_rgbd_camera"
+      use_nominal_extrinsics="${use_sim_time}">
+      <origin
+          xyz="${base_rgbd_x}
+              ${base_rgbd_y}
+              ${base_rgbd_z}"
+          rpy="${base_rgbd_R * deg_to_rad}
+              ${base_rgbd_P * deg_to_rad}
+              ${base_rgbd_Y * deg_to_rad}"/>
+    </xacro:sensor_d435i>
+    <!-- RGBD roof -->
+    <xacro:sensor_d435i
+      name="roof_rgbd_camera"
+      parent="base_link"
+      topics_ns="roof_rgbd_camera"
+      use_nominal_extrinsics="${use_sim_time}">
+      <origin
+          xyz="${roof_rgbd_x}
+              ${roof_rgbd_y}
+              ${roof_rgbd_z}"
+          rpy="${roof_rgbd_R * deg_to_rad}
+              ${roof_rgbd_P * deg_to_rad}
+              ${roof_rgbd_Y * deg_to_rad}"/>
+    </xacro:sensor_d435i>
+  </xacro:if>
 </robot>

File: omni_base_description/urdf/sensors/imu.urdf.xacro (robot description, xacro)
@@ -17,11 +17,5 @@
   <!-- MACRO DEFINITION -->
   <xacro:macro name="imu_sensor" params="name parent *origin update_rate">
-    <link name="${name}_link">
-      <inertial>
-        <mass value="0.01"/>
-        <origin xyz="0 0 0"/>
-        <inertia ixx="0.000001" ixy="0" ixz="0" iyy="0.000001" iyz="0" izz="0.000001"/>
-      </inertial>
-    </link>
+    <link name="${name}_link"/>
     <joint name="${name}_joint" type="fixed">
       <parent link="${parent}"/>

Commit message: Imported upstream version '2.12.0' of 'upstream'

File: omni_base_description/robots/omni_base.urdf.xacro (robot description, xacro)
@@ -24,5 +24,4 @@
   <!-- Execution env config -->
   <xacro:arg name="use_sim_time" default="false"/>
-  <xacro:arg name="is_multiple" default="false"/>
   <xacro:arg name="namespace" default=""/>
   <xacro:arg name="is_public_sim" default="false"/>
@@ -40,5 +39,5 @@
     <xacro:wrong_laser_model/>
   </xacro:if>
-  <xacro:if value="${add_on_module not in ['no-add-on', 'cobra']}">
+  <xacro:if value="${add_on_module not in ['no-add-on', 'cobra', 'horizon']}">
     <xacro:wrong_add_on_module/>
   </xacro:if>
@@ -48,5 +47,4 @@
   <!-- Execution env configuration -->
   <xacro:property name="use_sim_time" default="$(arg use_sim_time)"/>
-  <xacro:property name="is_multiple" value="$(arg is_multiple)" />
   <xacro:property name="namespace" value="$(arg namespace)" />
   <xacro:property name="is_public_sim" value="$(arg is_public_sim)" />
@@ -57,7 +55,12 @@
   <xacro:if value="${add_on_module == 'cobra'}">
     <xacro:include filename="$(find omni_base_description)/urdf/cameras_add_on/cameras_add_on.urdf.xacro" />
+    <xacro:cameras_add_on name="cameras_add_on" parent="base_link"/>
+  </xacro:if>
+  <xacro:if value="${add_on_module == 'horizon'}">
+    <xacro:include filename="$(find omni_base_description)/urdf/cameras_add_on/camera_horizon_add_on.urdf.xacro" />
+    <xacro:camera_horizon_add_on name="camera_horizon" parent="base_link"/>
   </xacro:if>
   <!-- Materials for visualization -->
-  <xacro:include filename="$(find pal_urdf_utils)/urdf/materials.urdf.xacro" />
+  <xacro:include filename="$(find pal_urdf_utils  )/urdf/materials.urdf.xacro" />
   <!-- Utils for degree to radian conversion -->
   <xacro:include filename="$(find pal_urdf_utils)/urdf/deg_to_rad.urdf.xacro" />
@@ -68,7 +71,3 @@
   <!-- Now we can start using the macros included above to define the actual robot -->
   <xacro:base_sensors name="base" front_laser_model="$(arg front_laser_model)" rear_laser_model="$(arg rear_laser_model)"/>
-  <!-- RGBD Sensors -->
-  <xacro:if value="${add_on_module == 'cobra'}">
-    <xacro:cameras_add_on name="cameras_add_on" parent="base_link"/>
-  </xacro:if>
 </robot>

File: omni_base_description/ros2_control/ros2_control.urdf.xacro (robot description, xacro)
@@ -15,5 +15,4 @@
   <!-- INCLUDES -->
   <xacro:include filename="$(find omni_base_description)/urdf/wheels/wheel.ros2_control.xacro"/>
-  <xacro:include filename="$(find omni_base_description)/urdf/sensors/sensors.ros2_control.xacro"/>
   <!-- MACRO DEFINITION-->
   <xacro:macro name="omni_base_ros2_control">
@@ -22,4 +21,9 @@
       <gazebo>
         <plugin filename="libgazebo_ros2_control.so" name="gazebo_ros2_control">
+          <ros>
+            <namespace>${namespace}</namespace>
+            <remapping>/tf:=tf</remapping>
+            <remapping>/tf_static:=tf_static</remapping>
+          </ros>
           <parameters>$(find omni_base_description)/ros2_control/gazebo_controller_manager_cfg.yaml</parameters>
           <!-- <robot_sim_type>gazebo_ros2_control/GazeboSystem</robot_sim_type>
@@ -36,6 +40,4 @@
           <plugin>gazebo_ros2_control/GazeboSystem</plugin>
         </hardware>
-        <!-- IMU sensor (only in simulation)-->
-        <xacro:ros2_control_imu name="base_imu_sensor"/>
       </xacro:if>
       <xacro:unless value="${use_sim_time}">

File: omni_base_description/urdf/base/base.gazebo.xacro (robot description, xacro)
@@ -34,4 +34,5 @@
       <plugin name="gazebo_ros_planar_move" filename="libgazebo_ros_planar_move.so">
         <ros>
+          <namespace>${namespace}</namespace>
           <remapping>cmd_vel:=mobile_base_controller/cmd_vel_unstamped</remapping>
           <remapping>odom:=mobile_base_controller/odom</remapping>
@@ -46,7 +47,4 @@
           <publish_odom_tf>false</publish_odom_tf>
         </xacro:unless>
-          <xacro:if value="${is_multiple}">
-            <namespace>/${nsp}</namespace>
-          </xacro:if>
         <odometry_frame>odom</odometry_frame>
         <robot_base_frame>base_footprint</robot_base_frame>

File: omni_base_description/urdf/base/base_sensors.urdf.xacro (robot description, xacro)
@@ -15,9 +15,9 @@
   <!-- INCLUDES -->
   <xacro:include filename="$(find omni_base_description)/urdf/base/base.urdf.xacro"/>
-  <xacro:include filename="$(find omni_base_description)/urdf/sensors/imu.urdf.xacro"/>
-  <xacro:include filename="$(find omni_base_description)/urdf/sensors/hokuyo_urg_04lx_ug01_laser.urdf.xacro"/>
-  <xacro:include filename="$(find omni_base_description)/urdf/sensors/sick_tim551_laser.urdf.xacro"/>
-  <xacro:include filename="$(find omni_base_description)/urdf/sensors/sick_tim561_laser.urdf.xacro"/>
-  <xacro:include filename="$(find omni_base_description)/urdf/sensors/sick_tim571_laser.urdf.xacro"/>
+  <xacro:include filename="$(find pal_urdf_utils)/urdf/interaction_sensors/imu.urdf.xacro"/>
+  <xacro:include filename="$(find pal_urdf_utils)/urdf/laser/hokuyo_urg_04lx_ug01_laser.urdf.xacro"/>
+  <xacro:include filename="$(find pal_urdf_utils)/urdf/laser/sick_tim551_laser.urdf.xacro"/>
+  <xacro:include filename="$(find pal_urdf_utils)/urdf/laser/sick_tim561_laser.urdf.xacro"/>
+  <xacro:include filename="$(find pal_urdf_utils)/urdf/laser/sick_tim571_laser.urdf.xacro"/>
   <!-- LASER MACRO DEFINITION -->
   <xacro:macro name="laser_sensor" params="name parent model ros_topic *origin update_rate:=10">

File: omni_base_description/urdf/cameras_add_on/cameras.urdf.xacro (robot description, xacro)
@@ -1,5 +1,5 @@
 <?xml version="1.0"?>
 <!--
-  Copyright (c) 2024 PAL Robotics S.L. All rights reserved.
+  Copyright (c) 2025 PAL Robotics S.L. All rights reserved.
   Licensed under the Apache License, Version 2.0 (the "License");
   you may not use this file except in compliance with the License.
@@ -26,7 +26,12 @@
   <xacro:property name="roof_rgbd_y" value="0.0"/>
   <xacro:property name="roof_rgbd_Y" value="0.0"/>
-  <!-- base/roof RGBD calibratable characteristics -->
-  <!-- spec = rgbd_z, rgbd_R and rgbd_P -->
-  <xacro:include filename="${calibration_path}/urdf/cameras_add_on/base_omni_base_calib.urdf.xacro"/>
+  <!-- RGBD base -->
+  <xacro:property name="base_rgbd_z" value="0.551436"/>
+  <xacro:property name="base_rgbd_R" value="0.0"/>
+  <xacro:property name="base_rgbd_P" value="55.0"/>
+  <!-- RGBD roof -->
+  <xacro:property name="roof_rgbd_z" value="0.483197"/>
+  <xacro:property name="roof_rgbd_R" value="0.0"/>
+  <xacro:property name="roof_rgbd_P" value="12.0"/>
   <xacro:include filename="$(find pal_urdf_utils)/urdf/deg_to_rad.urdf.xacro" />
   <xacro:if value="${camera_model == 'realsense-d435'}">

File: omni_base_description/urdf/cameras_add_on/cameras_add_on.urdf.xacro (robot description, xacro)
@@ -45,4 +45,4 @@
       </joint>
     </xacro:macro>
-    <xacro:include filename="$(find omni_base_description)/urdf/sensors/courier.urdf.xacro" />
+    <xacro:include filename="$(find omni_base_description)/urdf/cameras_add_on/cameras.urdf.xacro" />
   </robot>
