Commit message: Imported upstream version '2.14.1' of 'upstream'

File: omni_base_description/urdf/base/base.urdf.xacro (robot description, xacro)
@@ -20,5 +20,6 @@
   <xacro:property name="wheel_pair_separation" value="0.488"/>
   <xacro:property name="wheel_torque"     value="6.0"/>
-  <xacro:property name="wheel_velocity"   value="1.0"/>
+  <!-- TODO Compute real wheel max velocity -->
+  <xacro:property name="wheel_velocity"   value="100.0"/>
   <xacro:property name="suspension_sagital_separation" value="0.345"/>
   <!-- INCLUDES -->

File: omni_base_description/urdf/cameras_add_on/camera_horizon_add_on.urdf.xacro (robot description, xacro)
@@ -51,26 +51,24 @@
     </xacro:macro>
     <xacro:if value="${camera_model == 'realsense-d435'}">
-      <xacro:include filename="$(find realsense2_description)/urdf/_d435.urdf.xacro" />
-      <xacro:sensor_d435
+      <xacro:include filename="$(find pal_urdf_utils)/urdf/camera/realsense_d435.urdf.xacro" />
+      <xacro:realsense_d435
         name="rgbd_camera"
         parent="base_link"
-        topics_ns="rgbd_camera"
         use_nominal_extrinsics="${use_sim_time}">
         <origin
             xyz="${rgbd_x} ${rgbd_y} ${rgbd_z}"
             rpy="0.0 0.0 0.0"/>
-      </xacro:sensor_d435>
+      </xacro:realsense_d435>
     </xacro:if>
     <xacro:if value="${camera_model == 'realsense-d435i'}">
-      <xacro:include filename="$(find realsense2_description)/urdf/_d435i.urdf.xacro" />
-      <xacro:sensor_d435i
+      <xacro:include filename="$(find pal_urdf_utils)/urdf/camera/realsense_d435i.urdf.xacro" />
+      <xacro:realsense_d435i
         name="rgbd_camera"
         parent="base_link"
-        topics_ns="rgbd_camera"
         use_nominal_extrinsics="${use_sim_time}">
         <origin
             xyz="${rgbd_x} ${rgbd_y} ${rgbd_z}"
             rpy="0.0 0.0 0.0"/>
-      </xacro:sensor_d435i>
+      </xacro:realsense_d435i>
     </xacro:if>
   </robot>

File: omni_base_description/urdf/cameras_add_on/cameras.urdf.xacro (robot description, xacro)
@@ -37,10 +37,9 @@
   <xacro:if value="${camera_model == 'realsense-d435'}">
     <!-- INCLUDES -->
-    <xacro:include filename="$(find realsense2_description)/urdf/_d435.urdf.xacro" />
+    <xacro:include filename="$(find pal_urdf_utils)/urdf/camera/realsense_d435.urdf.xacro" />
     <!-- RGBD base -->
-    <xacro:sensor_d435
+    <xacro:realsense_d435
       name="base_rgbd_camera"
       parent="base_link"
-      topics_ns="base_rgbd_camera"
       use_nominal_extrinsics="${use_sim_time}">
       <origin
@@ -51,10 +50,9 @@
               ${base_rgbd_P * deg_to_rad}
               ${base_rgbd_Y * deg_to_rad}"/>
-    </xacro:sensor_d435>
+    </xacro:realsense_d435>
     <!-- RGBD roof -->
-    <xacro:sensor_d435
+    <xacro:realsense_d435
       name="roof_rgbd_camera"
       parent="base_link"
-      topics_ns="roof_rgbd_camera"
       use_nominal_extrinsics="${use_sim_time}">
       <origin
@@ -65,14 +63,13 @@
               ${roof_rgbd_P * deg_to_rad}
               ${roof_rgbd_Y * deg_to_rad}"/>
-    </xacro:sensor_d435>
+    </xacro:realsense_d435>
   </xacro:if>
   <xacro:if value="${camera_model == 'realsense-d435i'}">
     <!-- INCLUDES -->
-    <xacro:include filename="$(find realsense2_description)/urdf/_d435i.urdf.xacro" />
+    <xacro:include filename="$(find pal_urdf_utils)/urdf/camera/realsense_d435i.urdf.xacro" />
     <!-- RGBD base -->
-    <xacro:sensor_d435i
+    <xacro:realsense_d435i
       name="base_rgbd_camera"
       parent="base_link"
-      topics_ns="base_rgbd_camera"
       use_nominal_extrinsics="${use_sim_time}">
       <origin
@@ -83,10 +80,9 @@
               ${base_rgbd_P * deg_to_rad}
               ${base_rgbd_Y * deg_to_rad}"/>
-    </xacro:sensor_d435i>
+    </xacro:realsense_d435i>
     <!-- RGBD roof -->
-    <xacro:sensor_d435i
+    <xacro:realsense_d435i
       name="roof_rgbd_camera"
       parent="base_link"
-      topics_ns="roof_rgbd_camera"
       use_nominal_extrinsics="${use_sim_time}">
       <origin
@@ -97,5 +93,5 @@
               ${roof_rgbd_P * deg_to_rad}
               ${roof_rgbd_Y * deg_to_rad}"/>
-    </xacro:sensor_d435i>
+    </xacro:realsense_d435i>
   </xacro:if>
 </robot>

File: omni_base_description/urdf/wheels/wheel.ros2_control.xacro (robot description, xacro)
@@ -13,11 +13,9 @@
  -->
 <robot xmlns:xacro="http://ros.org/wiki/xacro">
+  <!-- TODO Compute real wheel max velocity -->
   <!-- MACRO DEFINITION -->
   <xacro:macro name="ros2_control_wheel" params="side">
     <joint name="wheel_${side}_joint">
-      <command_interface name="velocity">
-        <param name="min">-1</param>
-        <param name="max">1</param>
-      </command_interface>
+      <command_interface name="velocity"/>
       <state_interface name="position" />
     </joint>

File: omni_base_description/urdf/wheels/wheel.urdf.xacro (robot description, xacro)
@@ -87,5 +87,5 @@
       <child link="wheel_${side}_link" />
       <axis xyz="0 0 1" />
-      <limit effort="${torque}" velocity="${velocity / radius}"/>
+      <limit effort="${torque}" velocity="${velocity}"/>
       <dynamics damping="1.0" friction="2.0"/>
     </joint>
